Commit message: TP 6axis using ABB

File: reperes/tp_6axis/6axis/robot.urdf (robot description, URDF)
Before this commit: robot onshape, 33 links, 32 joints
Links:
- removed link component_base_1
- removed link component_base_1_1
- removed link component_base_1_2
- removed link component_base_1_3
- removed link component_base_1_4
- removed link component_p2_1
- removed link component_p2_1_1
- removed link component_p2_1_2
- removed link component_p2_1_3
- removed link component_p2_1_4
- removed link component_p2_1_5
- removed link component_p2_1_6
- removed link component_p2_1_7
- removed link component_p3_1
- removed link component_p3_1_1
- removed link component_p3_1_2
- removed link component_p3_1_3
- removed link component_p3_1_4
- removed link component_p3_1_5
- removed link component_p4_1
- removed link component_p4_1_1
- removed link component_p4_1_2
- removed link component_p4_1_3
- removed link component_p4_1_4
- removed link component_p5_1
- removed link component_p5_1_1
- removed link component_p5_1_2
- removed link component_p5_1_3
- removed link component_p5_1_4
- removed link p1_1
- removed link p1_1_1
- removed link p6_1
- removed link p6_1_1
- added link irb6620_220-150_m2004_rev0_01-1, mass 773.632; collision mesh filename=package:///irb6620_220-150_m2004_rev0_01-1.stl; visual mesh filename=package:///irb6620_220-150_m2004_rev0_01-1.stl
- added link irb6620_220-150_m2004_rev0_01-2, mass 641.051; collision mesh filename=package:///irb6620_220-150_m2004_rev0_01-2.stl; visual mesh filename=package:///irb6620_220-150_m2004_rev0_01-2.stl
- added link irb6620_220-150_m2004_rev0_01-3, mass 321.848; collision mesh filename=package:///irb6620_220-150_m2004_rev0_01-3.stl; visual mesh filename=package:///irb6620_220-150_m2004_rev0_01-3.stl
- added link irb6620_220-150_m2004_rev0_01-4, mass 390.365; collision mesh filename=package:///irb6620_220-150_m2004_rev0_01-4.stl; visual mesh filename=package:///irb6620_220-150_m2004_rev0_01-4.stl
- added link irb6620_220-150_m2004_rev0_01-5, mass 282.092; collision mesh filename=package:///irb6620_220-150_m2004_rev0_01-5.stl; visual mesh filename=package:///irb6620_220-150_m2004_rev0_01-5.stl
- added link irb6620_220-150_m2004_rev0_01-6, mass 48.6088; collision mesh filename=package:///irb6620_220-150_m2004_rev0_01-6.stl; visual mesh filename=package:///irb6620_220-150_m2004_rev0_01-6.stl
- added link irb6620_220-150_m2004_rev0_01-7, mass 7.065; collision mesh filename=package:///irb6620_220-150_m2004_rev0_01-7.stl; visual mesh filename=package:///irb6620_220-150_m2004_rev0_01-7.stl
Joints:
- removed joint component_base_1_1_fixing
- removed joint component_base_1_2_fixing
- removed joint component_base_1_3_fixing
- removed joint component_base_1_4_fixing
- removed joint component_p2_1_1_fixing
- removed joint component_p2_1_2_fixing
- removed joint component_p2_1_3_fixing
- removed joint component_p2_1_4_fixing
- removed joint component_p2_1_5_fixing
- removed joint component_p2_1_6_fixing
- removed joint component_p2_1_7_fixing
- removed joint component_p3_1_1_fixing
- removed joint component_p3_1_2_fixing
- removed joint component_p3_1_3_fixing
- removed joint component_p3_1_4_fixing
- removed joint component_p3_1_5_fixing
- removed joint component_p4_1_1_fixing
- removed joint component_p4_1_2_fixing
- removed joint component_p4_1_3_fixing
- removed joint component_p4_1_4_fixing
- removed joint component_p5_1_1_fixing
- removed joint component_p5_1_2_fixing
- removed joint component_p5_1_3_fixing
- removed joint component_p5_1_4_fixing
- removed joint motor1
- removed joint motor2
- removed joint motor3
- removed joint motor4
- removed joint motor5
- removed joint motor6
- removed joint p1_1_1_fixing
- removed joint p6_1_1_fixing
- added joint r1: type revolute, parent irb6620_220-150_m2004_rev0_01-1, child irb6620_220-150_m2004_rev0_01-2, origin xyz=3.19606e-34 6.95533e-18 0.23 rpy=-3.02406e-17 1.54074e-33 -4.27125e-50, axis 0 0 1, limit lower=-2.96706 upper=2.96706 effort=1 velocity=20
- added joint r2: type revolute, parent irb6620_220-150_m2004_rev0_01-2, child irb6620_220-150_m2004_rev0_01-3, origin xyz=0.32 -0.1305 0.45 rpy=-1.5708 -9.6472e-18 -6.93889e-15, axis 0 0 1, limit lower=-2.44346 upper=1.13446 effort=1 velocity=20
- added joint r3: type revolute, parent irb6620_220-150_m2004_rev0_01-3, child irb6620_220-150_m2004_rev0_01-4, origin xyz=-1.66533e-16 -0.975 -0.0955 rpy=6.48844e-17 2.91737e-34 0, axis 0 0 1, limit lower=-3.14159 upper=1.22173 effort=1 velocity=20
- added joint r4: type revolute, parent irb6620_220-150_m2004_rev0_01-4, child irb6620_220-150_m2004_rev0_01-5, origin xyz=0.182 -0.2 0.226 rpy=3.14159 -1.5708 0, axis 0 0 1, limit lower=-5.23599 upper=5.23599 effort=1 velocity=20
- added joint r5: type revolute, parent irb6620_220-150_m2004_rev0_01-5, child irb6620_220-150_m2004_rev0_01-6, origin xyz=-0.095 -2.22045e-16 0.705 rpy=-3.14159 -1.5708 0, axis 0 0 1, limit lower=-2.26893 upper=2.26893 effort=1 velocity=20
- added joint r6: type revolute, parent irb6620_220-150_m2004_rev0_01-6, child irb6620_220-150_m2004_rev0_01-7, origin xyz=0.163 -4.44089e-16 0.095 rpy=-3.14159 -1.5708 0, axis 0 0 1, limit lower=-5.23599 upper=5.23599 effort=1 velocity=20
